Commit message: The next commit

File: description/robot_core.xacro (robot description, xacro)
@@ -1,2 +1,77 @@
+<?xml version="1.0"?>
 <robot xmlns:xacro="http://www.ros.org/wiki/xacro">
+    <material name="white">
+        <color rgba="1 1 1 1"/>
+    </material>
+    <material name="orange">
+        <color rgba="1 0.3 0.1 1"/>
+    </material>
+    <material name="blue">
+        <color rgba="0.2 0.2 1 1"/>
+    </material>
+    <material name="black">
+        <color rgba="0 0 0 1"/>
+    </material>
+    <!-- BASE LINK-->
+    <link name="base_link">
+    </link>
+    <!--CHASSIS LINK-->
+    <joint name="chassis_joint" type="fixed">
+        <parent link="base_link"/>
+        <child link="chassis"/>
+        <origin xyz="-0.1 0 0"/>
+    </joint>"
+    <link name="chassis">
+        <visual>
+            <origin xyz="0.15 0 0.075"/>
+            <geometry>
+                <box size="0.3 0.3 0.15"/>
+            </geometry>
+            <material name="white"/>
+        </visual>
+    </link>
+    <!-- LEFT WHEEL LINK-->
+    <joint name="left_wheel_joint" type="continuous">
+        <parent link="base_link"/>
+        <child link="left_wheel"/>
+        <origin xyz="0 0.175 0" rpy="-${pi/2} 0 0"/>
+        <axis xyz="0 0 1"/>
+    </joint>
+    <link name="left_wheel">
+        <visual>
+            <geometry>
+                <cylinder radius="0.05" length="0.04"/>
+            </geometry>
+            <material name="blue"/>
+        </visual>
+    </link>
+    <!-- RIGHT WHEEL LINK-->
+    <joint name="right_wheel_joint" type="continuous">
+        <parent link="base_link"/>
+        <child link="right_wheel"/>
+        <origin xyz="0 -0.175 0" rpy="${pi/2} 0 0"/>
+        <axis xyz="0 0 -1"/>
+    </joint>
+    <link name="right_wheel">
+        <visual>
+            <geometry>
+                <cylinder radius="0.05" length="0.04"/>
+            </geometry>
+            <material name="blue"/>
+        </visual>
+    </link>
+    <!-- CASTOR WHEEL LINK-->
+     <joint name="castor_wheel_joint" type="fixed">
+        <parent link="chassis"/>
+        <child link="castor_wheel"/>
+        <origin xyz="0.24 0 0"/>
+    </joint>
+    <link name="castor_wheel">
+        <visual>
+            <geometry>
+                <sphere radius="0.05"/>
+            </geometry>
+            <material name="black"/>
+        </visual>
+        </link>
 </robot>

Commit message: URDF for the bto made

File: description/robot_core.xacro (robot description, xacro)
@@ -1,4 +1,5 @@
 <?xml version="1.0"?>
 <robot xmlns:xacro="http://www.ros.org/wiki/xacro">
+    <xacro:include filename="inertial_macros.xacro"/>
     <material name="white">
         <color rgba="1 1 1 1"/>
@@ -30,4 +31,13 @@
             <material name="white"/>
         </visual>
+        <collision>
+            <origin xyz="0.15 0 0.075"/>
+            <geometry>
+                <box size="0.3 0.3 0.15"/>
+            </geometry>
+        </collision>
+        <xacro:inertial_box mass="0.5" x="0.3" y="0.3" z="0">
+            <origin xyz="0.15 0 0.075" rpy="0 0 0"/>
+        </xacro:inertial_box>
     </link>
     <!-- LEFT WHEEL LINK-->
@@ -40,9 +50,19 @@
     <link name="left_wheel">
         <visual>
+            <origin xyz="0 0 0"/>
             <geometry>
+                <origin xyz="0 0 0"/>
                 <cylinder radius="0.05" length="0.04"/>
             </geometry>
             <material name="blue"/>
         </visual>
+        <collision>
+            <geometry>
+                <cylinder radius="0.05" length="0.04"/>
+            </geometry>
+        </collision>
+        <xacro:inertial_cylinder mass="0.1" length="0.04" radius="0.05">
+            <origin xyz="0 0 0" rpy="0 0 0"/>
+        </xacro:inertial_cylinder>
     </link>
     <!-- RIGHT WHEEL LINK-->
@@ -55,9 +75,18 @@
     <link name="right_wheel">
         <visual>
-            <geometry>
+            <origin xyz="0 0 0"/>
+            <geometry>        <origin xyz="0 0 0"/>
                 <cylinder radius="0.05" length="0.04"/>
             </geometry>
             <material name="blue"/>
         </visual>
+        <collision>
+            <geometry>
+                <cylinder radius="0.05" length="0.04"/>
+            </geometry>
+        </collision>
+        <xacro:inertial_cylinder mass="0.1" length="0.04" radius="0.05">
+            <origin xyz="0 0 0" rpy="0 0 0"/>
+        </xacro:inertial_cylinder>
     </link>
     <!-- CASTOR WHEEL LINK-->
@@ -69,4 +98,5 @@
     <link name="castor_wheel">
         <visual>
+            <origin xyz="0 0 0"/>
             <geometry>
                 <sphere radius="0.05"/>
@@ -74,4 +104,12 @@
             <material name="black"/>
         </visual>
-        </link>
+        <collision>
+            <geometry>
+                <sphere radius="0.05"/>
+            </geometry>
+        </collision>
+        <xacro:inertial_sphere mass="0.1" radius="0.05">
+            <origin xyz="0 0 0" rpy="0 0 0"/>
+        </xacro:inertial_sphere>
+    </link>
 </robot>

Commit message: Corrected URDF

File: description/robot_core.xacro (robot description, xacro)
@@ -22,5 +22,5 @@
         <child link="chassis"/>
         <origin xyz="-0.1 0 0"/>
-    </joint>"
+    </joint>
     <link name="chassis">
         <visual>
@@ -52,5 +52,4 @@
             <origin xyz="0 0 0"/>
             <geometry>
-                <origin xyz="0 0 0"/>
                 <cylinder radius="0.05" length="0.04"/>
             </geometry>
@@ -76,5 +75,5 @@
         <visual>
             <origin xyz="0 0 0"/>
-            <geometry>        <origin xyz="0 0 0"/>
+            <geometry>
                 <cylinder radius="0.05" length="0.04"/>
             </geometry>

Commit message: Commit

File: description/robot_core.xacro (robot description, xacro)
@@ -41,4 +41,7 @@
         </xacro:inertial_box>
     </link>
+    <gazebo reference="chassis">
+        <material>Gazebo/White</material>
+    </gazebo>
     <!-- LEFT WHEEL LINK-->
     <joint name="left_wheel_joint" type="continuous">
@@ -65,4 +68,7 @@
         </xacro:inertial_cylinder>
     </link>
+    <gazebo reference="left_wheel">
+        <material>Gazebo/Blue</material>
+    </gazebo>
     <!-- RIGHT WHEEL LINK-->
     <joint name="right_wheel_joint" type="continuous">
@@ -89,4 +95,7 @@
         </xacro:inertial_cylinder>
     </link>
+    <gazebo reference="right_wheel">
+        <material>Gazebo/Blue</material>
+    </gazebo>
     <!-- CASTOR WHEEL LINK-->
      <joint name="castor_wheel_joint" type="fixed">
@@ -112,3 +121,8 @@
         </xacro:inertial_sphere>
     </link>
+    <gazebo reference="castor_wheel">
+        <material>Gazebo/Black</material>
+        <mu1 value="0.001"/>
+        <mu2 value="0.001"/>
+    </gazebo>
 </robot>
